Commit message: add mesh and imu enable

File: flyingcar_description/urdf/flyingcar.gazebo.xacro (robot description, xacro)
@@ -7,3 +7,19 @@
     <material>Gazebo/Orange</material>
   </gazebo>
+  <gazebo>
+    <!--hector_gazebo_plugins-->
+    <plugin name="imu_controller" filename="libhector_gazebo_ros_imu.so">
+      <robotNamespace>/</robotNamespace>
+      <frameId>base_imu_link</frameId>
+      <updateRate>100.0</updateRate>
+      <bodyName>base_imu_link</bodyName>
+      <topicName>imu</topicName>
+      <accelDrift>0.005 0.005 0.005</accelDrift>
+      <accelGaussianNoise>0.005 0.005 0.005</accelGaussianNoise>
+      <rateDrift>0.005 0.005 0.005 </rateDrift>
+      <rateGaussianNoise>0.005 0.005 0.005 </rateGaussianNoise>
+      <headingDrift>0.005</headingDrift>
+      <headingGaussianNoise>0.005</headingGaussianNoise>
+    </plugin>
+  </gazebo>
 </robot>

File: flyingcar_description/urdf/sensors/_d435.urdf.xacro (robot description, xacro)
@@ -7,5 +7,5 @@
 -->
 <robot xmlns:xacro="http://ros.org/wiki/xacro">
-  <xacro:include filename="$(find ironfish_description)/urdf/sensors/_d435.gazebo.xacro"/>
+  <xacro:include filename="$(find flyingcar_description)/urdf/sensors/_d435.gazebo.xacro"/>
   <xacro:macro name="sensor_d435" params="parent *origin">
     <xacro:property name="M_PI" value="3.1415926535897931" />
@@ -41,5 +41,5 @@
         <geometry>
           <!-- <box size="${d435_cam_width} ${d435_cam_height} ${d435_cam_depth}"/> -->
-	  <mesh filename="package://ironfish_description/meshes/intel_realsense_d435/d435.dae" />
+	  <mesh filename="package://flyingcar_description/meshes/intel_realsense_d435/d435.dae" />
           <!--<mesh filename="package://realsense2_camera/meshes/d435/d435.dae" />-->
         </geometry>

File: flyingcar_description/urdf/sensors/hokuyo_utm30lx.gazebo.xacro (robot description, xacro)
@@ -19,5 +19,5 @@
           <range>
             <min>0.08</min>
-            <max>30.0</max>
+            <max>15.0</max>
             <resolution>0.01</resolution>
           </range>

File: flyingcar_description/urdf/sensors/hokuyo_utm30lx.urdf.xacro (robot description, xacro)
@@ -1,5 +1,5 @@
 <?xml version="1.0"?>
 <robot xmlns:xacro="http://ros.org/wiki/xacro">
-  <xacro:include filename="$(find ironfish_description)/urdf/sensors/hokuyo_utm30lx.gazebo.xacro" />
+  <xacro:include filename="$(find flyingcar_description)/urdf/sensors/hokuyo_utm30lx.gazebo.xacro" />
   <xacro:macro name="hokuyo_utm30lx" params="name parent *origin">
     <joint name="${name}_joint" type="fixed">
@@ -18,5 +18,5 @@
         <origin xyz="0 0 0" rpy="0 0 0" />
         <geometry>
-        <mesh filename="package://ironfish_description/meshes/hokuyo_utm30lx/hokuyo_utm_30lx.dae"/>
+        <mesh filename="package://flyingcar_description/meshes/hokuyo_utm30lx/hokuyo_utm_30lx.dae"/>
       </geometry>
       </visual>
@@ -29,34 +29,5 @@
     </link>
     <!-- extensions -->
-    <xacro:hokuyo_utm30lx_gazebo name="${name}" ros_topic="/scan" update_rate="40" ray_count="720" min_angle="-2" max_angle="2"/>
-  </xacro:macro>
-  <xacro:macro name="hokuyo_utm30lx_back" params="name parent">
-    <joint name="${name}_joint" type="fixed">
-      <!--origin xyz="0.105 0.000 0.229" rpy="0 0 0" /-->
-      <origin xyz="-0.180 0.006 0.0914430740677247" rpy="0 0 3.1415926535897931" />
-      <parent link="${parent}"/>
-      <child link="${name}_link"/>
-    </joint>
-    <link name="${name}_link">
-      <!--inertial>
-        <mass value="0.0000000270" />
-        <origin xyz="0 0 0" rpy="0 0 0" />
-        <inertia ixx="2.632e-4" ixy="0" ixz="0" iyy="2.632e-4" iyz="0" izz="2.632e-4" />
-      </inertial-->
-      <visual>
-        <origin xyz="0 0 0" rpy="0 0 0" />
-        <geometry>
-        <mesh filename="package://ironfish_description/meshes/hokuyo_utm30lx/hokuyo_utm_30lx.dae"/>
-      </geometry>
-      </visual>
-      <collision>
-        <origin xyz="0 0 0" rpy="0 0 0" />
-        <geometry>
-        <box size="0.058 0.058 0.087" />
-      </geometry>
-      </collision>
-    </link>
-    <!-- extensions -->
-    <xacro:hokuyo_utm30lx_gazebo name="${name}" ros_topic="/scan2" update_rate="40" ray_count="720" min_angle="-2" max_angle="2"/>
+    <xacro:hokuyo_utm30lx_gazebo name="${name}" ros_topic="/scan" update_rate="40" ray_count="720" min_angle="${-M_PI}" max_angle="${M_PI}"/>
   </xacro:macro>
 </robot>
