Commit message: correct the size in real world

File: flyingcar_description/urdf/flyingcar.urdf.xacro (robot description, xacro)
@@ -54,9 +54,9 @@
     <!-- Hokuyo utm30lx-->
     <xacro:hokuyo_utm30lx name="hokuyo" parent="${parent}">
-      <origin xyz="0.047 0.006 0.463" rpy="0 0 0"/> <!--real measure from blue extend version-->
+      <origin xyz="0.0 0.0 0.105" rpy="0 0 0"/> <!--real measure from blue extend version-->
     </xacro:hokuyo_utm30lx>
     <!-- Intel realsense-->
     <xacro:sensor_d435 parent="${parent}">
-      <origin xyz="0.047 0.006 0.463" rpy="0 0 0"/> <!--real measure from blue extend version-->
+      <origin xyz="0.032 0.0 0.05" rpy="0 0 0"/> <!--real measure from blue extend version-->
     </xacro:sensor_d435>
   </xacro:macro>

Commit message: fixed imu coordinate

File: flyingcar_description/urdf/flyingcar.urdf.xacro (robot description, xacro)
@@ -41,5 +41,5 @@
       <inertial>
         <mass value="0.001"/>
-        <origin rpy="0 0 0" xyz="0 0 0"/>
+        <origin rpy="0 3.1415 0" xyz="0 0 0"/>
         <inertia ixx="0.0001" ixy="0" ixz="0" iyy="0.000001" iyz="0" izz="0.0001"/>
       </inertial>

Commit message: fixed imu link coordinate z point down

File: flyingcar_description/urdf/flyingcar.urdf.xacro (robot description, xacro)
@@ -34,5 +34,5 @@
     <joint name="imu_joint" type="fixed">
       <axis xyz="0 0 0"/> <!-- 0 1 0 -->
-      <origin xyz="0 0 0.06"/>
+      <origin xyz="0 0 0.06" rpy="0 3.14159 0"/>
       <parent link="${parent}"/>
       <child link="base_imu_link"/>
@@ -41,5 +41,5 @@
       <inertial>
         <mass value="0.001"/>
-        <origin rpy="0 3.1415 0" xyz="0 0 0"/>
+        <origin rpy="0 0 0" xyz="0 0 0"/>
         <inertia ixx="0.0001" ixy="0" ixz="0" iyy="0.000001" iyz="0" izz="0.0001"/>
       </inertial>

Commit message: find the correct imu link setting

File: flyingcar_description/urdf/flyingcar.urdf.xacro (robot description, xacro)
@@ -34,5 +34,5 @@
     <joint name="imu_joint" type="fixed">
       <axis xyz="0 0 0"/> <!-- 0 1 0 -->
-      <origin xyz="0 0 0.06" rpy="0 3.14159 0"/>
+      <origin xyz="0 0 0.06" rpy="3.1416 0 3.1416"/>
       <parent link="${parent}"/>
       <child link="base_imu_link"/>

Commit message: correct the imu frame to the confirmed corrected pose

File: flyingcar_description/urdf/flyingcar.urdf.xacro (robot description, xacro)
@@ -34,5 +34,5 @@
     <joint name="imu_joint" type="fixed">
       <axis xyz="0 0 0"/> <!-- 0 1 0 -->
-      <origin xyz="0 0 0.06" rpy="3.1416 0 3.1416"/>
+      <origin xyz="0 0 0.06" rpy="0 3.1416 3.1416"/>
       <parent link="${parent}"/>
       <child link="base_imu_link"/>
