Commit message: fix material bug

File: flyingcar_description/robot/flyingcar_robot.urdf.xacro (robot description, xacro)
@@ -2,4 +2,5 @@
 <robot name="flyingcar" xmlns:xacro="https://www.ros.org/wiki/xacro" >
   <xacro:include filename="$(find flyingcar_description)/urdf/flyingcar.urdf.xacro" />
+  <xacro:include filename="$(find flyingcar_description)/urdf/flyingcar.materials.xacro"/>
   <xacro:flyingcar parent="base_link"/>
   <link name="base_link"><!--bottom of sensor pack-->

File: flyingcar_description/urdf/flyingcar.gazebo.xacro (robot description, xacro)
@@ -1,8 +1,5 @@
 <?xml version="1.0" ?>
 <robot name="flyingcar" xmlns:xacro="https://www.ros.org/wiki/xacro" >
-  <gazebo reference="base_link">
-    <material>Gazebo/Orange</material>
-  </gazebo>
-  <gazebo reference="body_link">
+  <gazebo reference="pack_link">
     <material>Gazebo/Orange</material>
   </gazebo>

File: flyingcar_description/urdf/flyingcar.urdf.xacro (robot description, xacro)
@@ -1,5 +1,4 @@
 <?xml version="1.0" ?>
 <robot xmlns:xacro="https://www.ros.org/wiki/xacro" >
-  <xacro:include filename="$(find flyingcar_description)/urdf/flyingcar.materials.xacro"/>
   <xacro:include filename="$(find flyingcar_description)/urdf/flyingcar.gazebo.xacro"/>
   <xacro:include filename="$(find flyingcar_description)/urdf/sensors/hokuyo_utm30lx.urdf.xacro" />
@@ -8,10 +7,10 @@
   <xacro:macro name="flyingcar" params="parent">
     <!--body of sensor-->
-    <joint name="body_link_joint" type="fixed">
+    <joint name="pack_link_joint" type="fixed">
       <origin xyz="0 0 0.0375" rpy="0 0 0"/>
       <parent link="${parent}"/>
-      <child link="body_link" />
+      <child link="pack_link" />
     </joint>
-    <link name="body_link">
+    <link name="pack_link">
       <inertial>
         <mass value="0.5"/>

Commit message: update description to real robot model

File: flyingcar_description/robot/flyingcar_robot.urdf.xacro (robot description, xacro)
@@ -4,12 +4,4 @@
   <xacro:include filename="$(find flyingcar_description)/urdf/flyingcar.materials.xacro"/>
   <xacro:flyingcar parent="base_link"/>
-  <link name="base_link"><!--bottom of sensor pack-->
-    <visual>
-      <origin xyz="0 0 0" rpy="0 0 0"/>
-      <geometry>
-        <box size="0.01 0.01 0.01" />
-      </geometry>
-      <material name="White" />
-    </visual>
-  </link>
+  <link name="base_link"/><!--bottom of sensor pack-->
 </robot>

File: flyingcar_description/urdf/flyingcar.urdf.xacro (robot description, xacro)
@@ -6,7 +6,7 @@
   <xacro:property name="M_PI" value="3.14159"/>
   <xacro:macro name="flyingcar" params="parent">
-    <!--body of sensor-->
+    <!--visual body of sensor-->
     <joint name="pack_link_joint" type="fixed">
-      <origin xyz="0 0 0.0375" rpy="0 0 0"/>
+      <origin xyz="0 0 0.04675" rpy="0 0 0"/>
       <parent link="${parent}"/>
       <child link="pack_link" />
@@ -20,5 +20,5 @@
       <collision name="collision_base_link">
         <geometry>
-          <box size="0.08 0.12 0.075"/>
+          <box size="0.08 0.12 0.0935"/>
         </geometry>
       </collision>
@@ -26,5 +26,5 @@
         <origin rpy="0 0 0" xyz="0 0 0"/>
         <geometry>
-          <box size="0.08 0.12 0.075"/>
+          <box size="0.08 0.12 0.0935"/>
         </geometry>
         <material name="blue"/>
@@ -34,5 +34,5 @@
     <joint name="imu_joint" type="fixed">
       <axis xyz="0 0 0"/> <!-- 0 1 0 -->
-      <origin xyz="0 0 0.06" rpy="0 3.1416 3.1416"/>
+      <origin xyz="0 0 0.078" rpy="0 3.1416 3.1416"/>
       <parent link="${parent}"/>
       <child link="base_imu_link"/>
@@ -44,18 +44,20 @@
         <inertia ixx="0.0001" ixy="0" ixz="0" iyy="0.000001" iyz="0" izz="0.0001"/>
       </inertial>
-      <visual>
-        <origin rpy="0 0 0" xyz="0 0 0"/>
-        <geometry>
-          <box size="0.001 0.001 0.001"/>
-        </geometry>
-      </visual>
     </link>
+    <!-- csi camera -->
+    <joint name="csi_camera_joint" type="fixed">
+      <axis xyz="0 0 0"/> <!-- 0 1 0 -->
+      <origin xyz="0 0 0.043" rpy="0 0 0"/>
+      <parent link="${parent}"/>
+      <child link="csi_camera_link"/>
+    </joint>
+    <link name="csi_camera_link"/>
     <!-- Hokuyo utm30lx-->
     <xacro:hokuyo_utm30lx name="hokuyo" parent="${parent}">
-      <origin xyz="0.0 0.0 0.105" rpy="0 0 0"/> <!--real measure from blue extend version-->
+      <origin xyz="0 0 0.1275" rpy="0 0 0"/> <!--real measure from blue extend version-->
     </xacro:hokuyo_utm30lx>
     <!-- Intel realsense-->
     <xacro:sensor_d435 parent="${parent}">
-      <origin xyz="0.032 0.0 0.05" rpy="0 0 0"/> <!--real measure from blue extend version-->
+      <origin xyz="0.032 0 0.071" rpy="0 0 0"/> <!--real measure from blue extend version-->
     </xacro:sensor_d435>
   </xacro:macro>
